File: analog-pid.kicad_sch (KiCad schematic)
At the start: 39 parts, among them J1 Conn_01x06_Socket, SW1 SS12D10, SW2 SS12D10, U1 MCP6004, U2 Opamp_Dual, U3 MCP6004, U4 NC7SZ86M5X

Commit message: Finished
Test points not needed.
Gonna skip the TVS diodes.
Finished decoupling caps.
Added rounded corners & mounting holes.
Parts:
- added C10, C9: 100nF, Capacitor_SMD:C_0805_2012Metric_Pad1.18x1.45mm_HandSolder, symbol Device:C
- U2: value Opamp_Dual -> TSV792IDT
- U5: value ~ -> TS5A4624
Connections:
- net +5V: now also C10.1, C9.1
- net GND: now also C10.2, C9.2

Commit message: finished
Parts:
- C2: value 6nF -> 100pF
- C3: value 2nF -> 1.5nF
- R12: value 1Meg -> 100k
- R13: value 100 -> 10k
- R15, R18: value 5k -> 1k
- R16, R17: value 5k -> 10k
- R5: value 2k -> 1Meg
- R6: value 2k -> 10k
Changed lines of the file:
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@@
 			)
 		)
-		(property "Value" "5k"
+		(property "Value" "10k"
 			(at 123.19 138.43 90)
 			(effects
@@
 			)
 		)
-		(property "Value" "100"
+		(property "Value" "10k"
 			(at 81.28 163.83 90)
 			(effects
@@
 			)
 		)
-		(property "Value" "2k"
+		(property "Value" "10k"
 			(at 29.21 175.26 90)
 			(effects
@@
 			)
 		)
-		(property "Value" "1Meg"
+		(property "Value" "100k"
 			(at 93.98 163.83 90)
 			(effects
@@
 			)
 		)
-		(property "Value" "5k"
+		(property "Value" "1k"
 			(at 134.62 128.27 90)
 			(effects
@@
 			)
 		)
-		(property "Value" "5k"
+		(property "Value" "1k"
 			(at 134.62 90.17 90)
 			(effects
@@
 			)
 		)
-		(property "Value" "2nF"
+		(property "Value" "1.5nF"
 			(at 43.18 173.99 90)
 			(effects
@@
 			)
 		)
-		(property "Value" "6nF"
+		(property "Value" "100pF"
 			(at 58.42 157.48 90)
 			(effects
@@
 			)
 		)
-		(property "Value" "5k"
+		(property "Value" "10k"
 			(at 123.19 100.33 90)
 			(effects
@@
 			)
 		)
-		(property "Value" "2k"
+		(property "Value" "1Meg"
 			(at 58.42 171.45 90)
 			(effects
